File: Hardware/SparkX_EZ_ZOE-M8Q.brd (EAGLE design)
At the start: 10.7 x 40.6 mm, 50 parts, among them J4 U.FL, Q2 20V/4.2A/52mΩ/1.4W, U1 UBLOX_ZOE_M8-0-10, X1 32.768kHz

Commit message: Review updates
Parts:
- added U$12: (no value), output:#IN#0
- added U$13: (no value), output:#OUT#0
- Q2: device SparkFun-DiscreteSemi:SOT23-3@1 -> SparkFun-DiscreteSemi:SOT23-3
- U1: value UBLOX_ZOE_M8-0-10 -> U-BLOX_ZOE_M8Q-0-10
- moved LOGO2 13.2 mm to (1.91, 19.1)
- moved L1 0.44 mm to (2.16, 24.8)
Connections:
- net V_BATT renamed PROC_PWR_EN
- net !SAFEBOOT!: now also !SAFEBOOT!.1; no longer !SAFEBOOT!.P$1
- net GPIO0: now also GPIO0.1; no longer GPIO0.P$1
- net RXD: now also RXD.1; no longer RXD.P$1
- net TXD: now also TXD.1; no longer TXD.P$1
- net VDD: now also VDD.1; no longer VDD.P$1
- net V_BCKP: now also V_BCKP.1; no longer V_BCKP.P$1
